File: hardware/design/cicada-main/cicada-main.kicad_pcb (KiCad board)
At the start: 2 copper layers, 41.7 x 58.7 mm, 31 parts, among them U1 ESP-07, X1 Expansion slot 1, X2 Expansion slot 2, X3 Escaper, X4 UART

Commit message: added new board cicada-main-v4
Parts:
- removed C4: 20 uF, Capacitor_SMD:C_1206_3216Metric_Pad1.42x1.75mm_HandSolder
- removed D2: MT3608, Package_TO_SOT_SMD:SOT-23-6_Handsoldering
- removed L1: SPM4020T-4R7, custom:SPM4020T
- removed R10, R9: 3k3, Resistor_SMD:R_0805_2012Metric_Pad1.15x1.40mm_HandSolder
- removed R11: 160k, Resistor_SMD:R_0805_2012Metric_Pad1.15x1.40mm_HandSolder
- removed R12: 22k, Resistor_SMD:R_0805_2012Metric_Pad1.15x1.40mm_HandSolder
- removed R7, R8: 1k2, Resistor_SMD:R_0805_2012Metric_Pad1.15x1.40mm_HandSolder
- removed VD1: SS34, Diode_SMD:D_SMA_Handsoldering
- added X5: Ext Pwr, Connector_Molex:Molex_PicoBlade_53047-0410_1x02_P1.25mm_Vertical, F.Cu at (140.3, 107.4)
- C1: footprint Capacitor_SMD:C_0805_2012Metric_Pad1.15x1.40mm_HandSolder -> Capacitor_SMD:C_0805_2012Metric; moved to F.Cu
- C2, C3: footprint Capacitor_SMD:C_1206_3216Metric_Pad1.42x1.75mm_HandSolder -> Capacitor_SMD:C_1206_3216Metric
- D1: value LM1117-3.3 -> LDL1117SR33
- JP1: footprint Connector_PinHeader_2.54mm:PinHeader_1x03_P2.54mm_Vertical -> Jumper:SolderJumper-3_P1.3mm_Open_Pad1.0x1.5mm
- JP2: value Sold for 1S Battery -> Jumper_3_Bridged12; footprint Resistor_SMD:R_0805_2012Metric -> Jumper:SolderJumper-3_P1.3mm_Open_Pad1.0x1.5mm
- R1: value 160k -> 3k3; footprint Resistor_SMD:R_0805_2012Metric_Pad1.15x1.40mm_HandSolder -> Resistor_SMD:R_0805_2012Metric; moved to F.Cu
- R2: value 33k -> 3k3; footprint Resistor_SMD:R_0805_2012Metric_Pad1.15x1.40mm_HandSolder -> Resistor_SMD:R_0805_2012Metric; moved to F.Cu
- R3, R4, R5: footprint Resistor_SMD:R_0805_2012Metric_Pad1.15x1.40mm_HandSolder -> Resistor_SMD:R_0805_2012Metric
- R6: footprint Resistor_SMD:R_0805_2012Metric_Pad1.15x1.40mm_HandSolder -> Resistor_SMD:R_0805_2012Metric; moved to F.Cu
- X3: value Escaper -> ESC; footprint Connector_PinHeader_2.54mm:PinHeader_1x06_P2.54mm_Vertical -> Connector_Molex:Molex_PicoBlade_53047-1610_1x08_P1.25mm_Vertical
- X4: value UART -> GPS; footprint Connector_PinHeader_2.54mm:PinHeader_1x04_P2.54mm_Vertical -> Connector_Molex:Molex_PicoBlade_53047-1210_1x06_P1.25mm_Vertical
- moved R3 27.5 mm to (149.6, 99.5)
- moved R4 27.2 mm to (152.4, 90.7), turned to 270 degrees
- moved R5 20.6 mm to (134.0, 95.8), turned to 0 degrees
- moved R6 6.85 mm to (147.8, 95.8), turned to 0 degrees
- moved R1 5.23 mm to (128.4, 81.8), turned to 0 degrees
- moved JP1 2.54 mm to (141.0, 95.8), turned to 0 degrees
- moved JP2 2.04 mm to (138.3, 114.0)
- moved X3 2.03 mm to (136.7, 118.1), turned to 0 degrees
- moved R2 1.50 mm to (128.4, 77.7), turned to 0 degrees
- moved X4 0.95 mm to (144.1, 99.6), turned to 180 degrees
- moved C2 0.70 mm to (133.4, 99.6), turned to 0 degrees
- moved C3 0.21 mm to (133.6, 114.0)
- moved C1 0.08 mm to (129.5, 92.6)
Connections:
- C3 pad 1: +5V -> Net-(C3-Pad1)
- D1 pad 3: +5V -> Net-(C3-Pad1)
- JP2 pad 2: Net-(C4-Pad1) -> Net-(C3-Pad1)
- R1 pad 1: +BATT -> +3V3
- R1 pad 2: ADC -> Net-(R1-Pad2)
- R2 pad 1: ADC -> +3V3
- R2 pad 2: GNDD -> Net-(R2-Pad2)
- R3 pad 2: Net-(R3-Pad2) -> /M2
- R4 pad 1: +3V3 -> /M1
- R4 pad 2: Net-(R4-Pad2) -> GNDD
- R5 pad 2: /M2 -> Net-(JP1-Pad1)
- R6 pad 1: /M1 -> Net-(JP1-Pad3)
- U1 pad 1: Net-(R4-Pad2) -> Net-(R2-Pad2)
- U1 pad 2: ADC -> /ADC
- U1 pad 3: Net-(R3-Pad2) -> Net-(R1-Pad2)
- X1 pad 2: ADC -> /ADC
- X1 pad 3: +5V -> /CURN
- X4 pad 1: +3V3 -> +5V
- X4 pad 2: /RXD -> /TXD
- X4 pad 3: /TXD -> /RXD
- X4 pad 4: GNDD -> /SCL
Routing:
- net GNDD: track 134.4 -> 9.96 mm, vias 8 -> 4
- net /CURN: track 0.00 -> 60.8 mm
- net +5V: track 61.7 -> 16.3 mm, vias 1 -> 0
- net /SDA: track 10.5 -> 44.5 mm, vias 0 -> 1
- net +3V3: track 89.8 -> 58.3 mm, vias 3 -> 1
- net /SCL: track 13.0 -> 43.8 mm, vias 0 -> 1
- net Net-(C4-Pad1): track 17.4 -> 0.00 mm
- net /ADC: track 0.00 -> 10.5 mm
- net ADC: track 9.46 -> 0.00 mm
- net /M1: track 42.0 -> 50.9 mm
- net Net-(D2-Pad1): track 8.88 -> 0.00 mm
- net Net-(C3-Pad1): track 0.00 -> 8.18 mm
- net +BATT: track 67.8 -> 62.0 mm, vias 1 -> 0
- net /M4: track 56.8 -> 61.7 mm
- net /M3: track 85.1 -> 89.9 mm, vias 0 -> 1
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Other:
- outline, holes or cut-outs redrawn
- net class Default: clearance 0.4 -> 0.2; via_dia 1.6 -> 1.1; via_drill 0.7 -> 0.5
- net class power: clearance 0.4 -> 0.2; via_dia 1.6 -> 1.1; via_drill 0.7 -> 0.5
- rule trace_clearance: 0.4 -> 0.2
- board text added: "+"
- board text added: "-"
- board text added: "1"
- board text added: "2"
- board text added: "3"
- board text added: "4"
- board text added: "C"
- board text added: "D"
- board text added: "Ext Pwr 5V"
- board text added: "Prog"
- board text added: "R"
- board text added: "T"
- board text removed: "BN180"
- board text removed: "prog"
