File: hardware/design/cicada-main/cicada-main.sch (KiCad schematic (older format))
At the start: 27 parts, among them U1 ESP-07, X1 Expansion slot 1, X2 Expansion slot 2, X3 Escaper, X4 UART

Commit message: added new board cicada-main-v4
Parts:
- removed C4: 20 uF, Capacitor_SMD:C_1206_3216Metric_Pad1.42x1.75mm_HandSolder, symbol Device:C
- removed D2: MT3608, Package_TO_SOT_SMD:SOT-23-6_Handsoldering, symbol mt3608:MT3608
- removed JP2: Sold for 1S Battery, Resistor_SMD:R_0805_2012Metric, symbol Jumper:Jumper_2_Open
- removed L1: SPM4020T-4R7, custom:SPM4020T, symbol pspice:INDUCTOR
- removed R1, R11: 160k, Resistor_SMD:R_0805_2012Metric_Pad1.15x1.40mm_HandSolder, symbol Device:R
- removed R12: 22k, Resistor_SMD:R_0805_2012Metric_Pad1.15x1.40mm_HandSolder, symbol Device:R
- removed R2: 33k, Resistor_SMD:R_0805_2012Metric_Pad1.15x1.40mm_HandSolder, symbol Device:R
- removed R7, R8: 3k6, Resistor_SMD:R_0805_2012Metric_Pad1.15x1.40mm_HandSolder, symbol Device:R
- removed VD1: SS34, Diode_SMD:D_SMA_Handsoldering, symbol Device:D_Schottky
- removed X3: Escaper, Connector_PinHeader_2.54mm:PinHeader_1x06_P2.54mm_Vertical, symbol Connector_Generic:Conn_01x06
- removed X4: UART, Connector_PinHeader_2.54mm:PinHeader_1x04_P2.54mm_Vertical, symbol Connector_Generic:Conn_01x04
- added JP2: Jumper_3_Bridged12, Jumper:SolderJumper-3_P1.3mm_Open_Pad1.0x1.5mm, symbol Jumper:Jumper_3_Bridged12
- added X3: ESC, Connector_Molex:Molex_PicoBlade_53047-1610_1x08_P1.25mm_Vertical, symbol Connector_Generic:Conn_01x08
- added X4: GPS, Connector_Molex:Molex_PicoBlade_53047-1210_1x06_P1.25mm_Vertical, symbol Connector_Generic:Conn_01x06
- added X5: Ext Pwr, Connector_Molex:Molex_PicoBlade_53047-0410_1x02_P1.25mm_Vertical, symbol Connector_Generic:Conn_01x02
- C1: footprint Capacitor_SMD:C_0805_2012Metric_Pad1.15x1.40mm_HandSolder -> Capacitor_SMD:C_0805_2012Metric
- C2, C3: footprint Capacitor_SMD:C_1206_3216Metric_Pad1.42x1.75mm_HandSolder -> Capacitor_SMD:C_1206_3216Metric
- D1: value LM1117-3.3 -> LDL1117SR33
- JP1: footprint Connector_PinHeader_2.54mm:PinHeader_1x03_P2.54mm_Vertical -> Jumper:SolderJumper-3_P1.3mm_Open_Pad1.0x1.5mm
- R1: renamed from R3; footprint Resistor_SMD:R_0805_2012Metric_Pad1.15x1.40mm_HandSolder -> Resistor_SMD:R_0805_2012Metric
- R2: renamed from R4; footprint Resistor_SMD:R_0805_2012Metric_Pad1.15x1.40mm_HandSolder -> Resistor_SMD:R_0805_2012Metric
- R3: renamed from R5; footprint Resistor_SMD:R_0805_2012Metric_Pad1.15x1.40mm_HandSolder -> Resistor_SMD:R_0805_2012Metric
- R4: renamed from R6; footprint Resistor_SMD:R_0805_2012Metric_Pad1.15x1.40mm_HandSolder -> Resistor_SMD:R_0805_2012Metric
- R5: renamed from R9; footprint Resistor_SMD:R_0805_2012Metric_Pad1.15x1.40mm_HandSolder -> Resistor_SMD:R_0805_2012Metric
- R6: renamed from R10; footprint Resistor_SMD:R_0805_2012Metric_Pad1.15x1.40mm_HandSolder -> Resistor_SMD:R_0805_2012Metric
Connections:
- net +5V: now also JP2.3 (B), X4.1 (Pin_1), X5.1 (Pin_1); no longer C3.1, D1.3 (VI), X1.3 (Pin_3)
- net +BATT: now also JP2.1 (A), X3.2 (Pin_2)
- net GNDD: now also X3.1 (Pin_1), X4.6 (Pin_6), X5.2 (Pin_2)
- net M1: now also X3.6 (Pin_6)
- net M2: now also X3.5 (Pin_5)
- net M3: now also X3.4 (Pin_4)
- net M4: now also X3.3 (Pin_3)
- net RXD: now also X4.3 (Pin_3)
- net SCL: now also X4.4 (Pin_4)
- net SDA: now also X4.5 (Pin_5)
- net TXD: now also X4.2 (Pin_2)
- new net: C3.1, D1.3 (VI), JP2.2 (C)
- new net CURN: X1.3 (Pin_3), X3.7 (Pin_7)
- no-connect marks 0 -> 1
Other:
- note added: "1. Sold pin1+pin2 of JP2 to power from 1S LiPo\n2. Sold pin2+pin3 of JP2 to power from external 5V\n3. Don't mount LM1117 or AMS1117 - they have big\n dropout voltage\n4. Mount LDL1117SR33 from STMicroelectronics\n5. Don't mount pull up resistors bigger 3k3\n it causes a problem to upload firmware by UART"
- note removed: "3V3"
- note removed: "GND"
- note removed: "RXD"
- note removed: "TXD"
- moved on the sheet: C1, C2, C3, D1, JP1, R1, R2, R3, R4, R5, R6, U1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
